Commit message: add serial port

File: ros2_control_demo_description/diffbot_description/ros2_control/diffbot.ros2_control.xacro (robot description, xacro)
@@ -5,5 +5,5 @@
       <hardware>
         <plugin>ros2_control_demo_hardware/DiffBotSystemHardware</plugin>
-        <param name="example_param_hw_start_duration_sec">0</param>
+        <param name="ddms_tty">/dev/ttyACM0</param>
         <param name="example_param_hw_stop_duration_sec">3.0</param>
       </hardware>

File: ros2_control_demo_description/diffbot_description/urdf/diffbot_description.urdf.xacro (robot description, xacro)
@@ -4,12 +4,12 @@
   <!-- Constants for robot dimensions -->
   <xacro:property name="PI" value="3.1415926535897931"/>
-  <xacro:property name="base_mass" value="0.4" /> <!-- arbitrary value for base mass -->
-  <xacro:property name="base_width" value="0.2" />
+  <xacro:property name="base_mass" value="0.5" /> <!-- arbitrary value for base mass -->
+  <xacro:property name="base_width" value="0.178" />
   <xacro:property name="base_length" value="0.2" />
   <xacro:property name="base_height" value="0.05" />
   <xacro:property name="wheel_mass" value="0.5" /> <!-- arbitrary value for wheel mass -->
-  <xacro:property name="wheel_len" value="0.020" />
+  <xacro:property name="wheel_len" value="0.0428" />
   <xacro:property name="wheel_radius" value="0.05125" />
-  <xacro:property name="wheel_offset_y" value="0.089" />
+  <xacro:property name="wheel_offset_y" value="0.1115" />
   <xacro:property name="caster_wheel_mass" value="0.2" /> <!-- arbitrary value for caster wheel mass -->
   <xacro:property name="caster_wheel_radius" value="0.058" />
@@ -19,23 +19,26 @@
     <collision>
       <origin xyz="0 0 0" rpy="0 0 0"/>
-      <geometry>
-        <box size="${base_width} ${base_length} ${base_height}"/>
-      </geometry>
     </collision>
-    <visual>
-      <origin xyz="0 0 ${base_height/2}" rpy="0 0 0"/>
-      <geometry>
-        <box size="${base_width} ${base_length} ${base_height}"/>
-      </geometry>
-      <material name="orange"/>
-    </visual>
-    <inertial>
-      <origin xyz="0 0 0" rpy="0 0 0"/>
-      <mass value="${base_mass}"/>
-      <inertia
-        ixx="${base_mass / 12.0 * (base_length*base_length + base_height*base_height)}" ixy="0.0" ixz="0.0"
-        iyy="${base_mass / 12.0 * (base_height*base_height + base_width*base_width)}" iyz="0.0"
-        izz="${base_mass / 12.0 * (base_width*base_width + base_length*base_length)}"/>
-      </inertial>
+  </link>
+      <joint name="${prefix}base_joint" type="fixed">
+      <parent link="${prefix}base_link"/>
+      <child link="${prefix}base_platform"/>
+      <origin xyz="${-base_width/2} 0 ${base_height/2}" rpy="0 0 0"/>
+      <axis xyz="0 0 0"/>
+    </joint>
+    <link name="${prefix}base_platform">
+      <collision>
+        <origin xyz="0 0 ${base_height/2}" rpy="0 0 0"/>
+        <geometry>
+          <box size="${base_width} ${base_length} ${base_height}"/>
+        </geometry>
+      </collision>
+      <visual>
+        <origin xyz="0 0 ${base_height/2}" rpy="0 0 0"/>
+        <geometry>
+          <box size="${base_width} ${base_length} ${base_height}"/>
+        </geometry>
+        <material name="orange"/>
+      </visual>
     </link>
     <joint name="${prefix}left_wheel_joint" type="continuous">
@@ -101,37 +104,8 @@
         </inertial>
       </link>
-    <joint name="${prefix}caster_frontal_wheel_joint" type="fixed">
-      <parent link="${prefix}base_link"/>
-      <child link="${prefix}caster_frontal_wheel"/>
-      <origin xyz="${base_width/2 - caster_wheel_radius} 0 ${z_offset}" rpy="0 0 0"/>
-    </joint>
-    <!-- caster frontal wheel Link -->
-    <link name="${prefix}caster_frontal_wheel">
-      <collision>
-        <origin xyz="0 0 0" rpy="0 0 0"/>
-        <geometry>
-          <sphere radius="${caster_wheel_radius}"/>
-        </geometry>
-      </collision>
-      <visual>
-        <origin xyz="0 0 0" rpy="0 0 0"/>
-        <geometry>
-          <sphere radius="${caster_wheel_radius}"/>
-        </geometry>
-        <material name="white"/>
-      </visual>
-      <inertial>
-        <origin xyz="0 0 0" rpy="0 0 0"/>
-        <mass value="${caster_wheel_mass}"/>
-        <inertia
-          ixx="${caster_wheel_mass * 0.4 * (caster_wheel_radius * caster_wheel_radius)}" ixy="0.0" ixz="0.0"
-          iyy="${caster_wheel_mass * 0.4 * (caster_wheel_radius * caster_wheel_radius)}" iyz="0.0"
-          izz="${caster_wheel_mass * 0.4 * (caster_wheel_radius * caster_wheel_radius)}"/>
-        </inertial>
-      </link>
     <joint name="${prefix}caster_rear_wheel_joint" type="fixed">
       <parent link="${prefix}base_link"/>
       <child link="${prefix}caster_rear_wheel"/>
-      <origin xyz="${-base_width/2 + caster_wheel_radius} 0 ${z_offset}" rpy="0 0 0"/>
+      <origin xyz="${-base_width + caster_wheel_radius} 0 ${z_offset}" rpy="0 0 0"/>
     </joint>
     <!-- caster rear wheel Link -->

File: ros2_control_demo_description/diffbot_description/urdf/diffbot_system.urdf.xacro (robot description, xacro)
@@ -8,5 +8,5 @@
   <xacro:arg name="use_gazebo" default="false" />
   <!-- Enable setting arguments from the launch file -->
-  <xacro:arg name="use_fake_hardware" default="true" />
+  <xacro:arg name="use_fake_hardware" default="false" />
   <xacro:arg name="mock_sensor_commands" default="false" />
   <xacro:arg name="prefix" default="" />
