Commit message: add serial port

File: ros2_control_demo_description/diffbot_description/urdf/diffbot_description.urdf.xacro (robot description, xacro)
@@ -4,13 +4,14 @@
   <!-- Constants for robot dimensions -->
   <xacro:property name="PI" value="3.1415926535897931"/>
-  <xacro:property name="base_mass" value="0.3" /> <!-- arbitrary value for base mass -->
-  <xacro:property name="base_width" value="0.1" />
-  <xacro:property name="base_length" value="0.1" />
+  <xacro:property name="base_mass" value="0.4" /> <!-- arbitrary value for base mass -->
+  <xacro:property name="base_width" value="0.2" />
+  <xacro:property name="base_length" value="0.2" />
   <xacro:property name="base_height" value="0.05" />
-  <xacro:property name="wheel_mass" value="0.3" /> <!-- arbitrary value for wheel mass -->
+  <xacro:property name="wheel_mass" value="0.5" /> <!-- arbitrary value for wheel mass -->
   <xacro:property name="wheel_len" value="0.020" />
-  <xacro:property name="wheel_radius" value="0.015" />
-  <xacro:property name="caster_wheel_mass" value="0.1" /> <!-- arbitrary value for caster wheel mass -->
-  <xacro:property name="caster_wheel_radius" value="0.015" />
+  <xacro:property name="wheel_radius" value="0.05125" />
+  <xacro:property name="wheel_offset_y" value="0.089" />
+  <xacro:property name="caster_wheel_mass" value="0.2" /> <!-- arbitrary value for caster wheel mass -->
+  <xacro:property name="caster_wheel_radius" value="0.058" />
   <xacro:property name="z_offset" value="-${base_height/2}" /> <!-- Space btw top of beam and the each joint -->
   <!-- Base Link -->
@@ -41,5 +42,5 @@
       <parent link="${prefix}base_link"/>
       <child link="${prefix}left_wheel"/>
-      <origin xyz="0 -${base_width/2} ${z_offset}" rpy="0 0 0"/>
+      <origin xyz="0 -${wheel_offset_y} ${z_offset}" rpy="0 0 0"/>
       <axis xyz="0 1 0"/>
       <dynamics damping="0.2"/>
@@ -72,5 +73,5 @@
       <parent link="${prefix}base_link"/>
       <child link="${prefix}right_wheel"/>
-      <origin xyz="0 ${base_width/2} ${z_offset}" rpy="0 0 0"/>
+      <origin xyz="0 ${wheel_offset_y} ${z_offset}" rpy="0 0 0"/>
       <axis xyz="0 1 0"/>
       <dynamics damping="0.2"/>

Commit message: localization ok, nav and slam next

File: ros2_control_demo_description/diffbot_description/urdf/diffbot_description.urdf.xacro (robot description, xacro)
@@ -2,4 +2,6 @@
 <robot xmlns:xacro="http://www.ros.org/wiki/xacro">
   <xacro:macro name="diffbot" params="prefix">
+  <xacro:include filename="/home/mg/ros2_ddws/install/realsense2_description/share/realsense2_description/urdf/_d435i.urdf.xacro"/>
+  <xacro:include filename="/home/mg/ros2_ddws/install/realsense2_description/share/realsense2_description/urdf/_d435i_imu_modules.urdf.xacro"/>
   <!-- Constants for robot dimensions -->
   <xacro:property name="PI" value="3.1415926535897931"/>
@@ -13,37 +15,39 @@
   <xacro:property name="wheel_offset_y" value="0.1115" />
   <xacro:property name="caster_wheel_mass" value="0.2" /> <!-- arbitrary value for caster wheel mass -->
-  <xacro:property name="caster_wheel_radius" value="0.058" />
+  <xacro:property name="caster_wheel_radius" value="0.033" />
   <xacro:property name="z_offset" value="-${base_height/2}" /> <!-- Space btw top of beam and the each joint -->
-  <!-- Base Link -->
+  <!-- *********************** Base Link *********************** -->
   <link name="${prefix}base_link">
-    <collision>
-      <origin xyz="0 0 0" rpy="0 0 0"/>
-    </collision>
   </link>
       <joint name="${prefix}base_joint" type="fixed">
       <parent link="${prefix}base_link"/>
       <child link="${prefix}base_platform"/>
-      <origin xyz="${-base_width/2} 0 ${base_height/2}" rpy="0 0 0"/>
+      <origin xyz="${-base_length/2} 0 ${wheel_radius}" rpy="0 0 0"/>
       <axis xyz="0 0 0"/>
     </joint>
     <link name="${prefix}base_platform">
       <collision>
-        <origin xyz="0 0 ${base_height/2}" rpy="0 0 0"/>
+        <origin xyz="0 0 0" rpy="0 0 0"/>
         <geometry>
-          <box size="${base_width} ${base_length} ${base_height}"/>
+          <box size="${base_length} ${base_width} ${base_height}"/>
         </geometry>
       </collision>
       <visual>
-        <origin xyz="0 0 ${base_height/2}" rpy="0 0 0"/>
+        <origin xyz="0 0 0" rpy="0 0 0"/>
         <geometry>
-          <box size="${base_width} ${base_length} ${base_height}"/>
+          <box size="${base_length} ${base_width} ${base_height}"/>
         </geometry>
         <material name="orange"/>
       </visual>
     </link>
+<!-- *********************** d435i *********************** -->
+  <xacro:sensor_d435i parent="base_link" use_nominal_extrinsics="false">
+    <origin xyz="0 0 ${wheel_radius}" rpy="0 0 0"/>
+  </xacro:sensor_d435i>
+<!-- *********************** caster rear wheel Link *********************** -->
     <joint name="${prefix}left_wheel_joint" type="continuous">
       <parent link="${prefix}base_link"/>
       <child link="${prefix}left_wheel"/>
-      <origin xyz="0 -${wheel_offset_y} ${z_offset}" rpy="0 0 0"/>
+      <origin xyz="0 -${wheel_offset_y} ${wheel_radius}" rpy="${PI/2} 0 0"/>
       <axis xyz="0 1 0"/>
       <dynamics damping="0.2"/>
@@ -52,5 +56,5 @@
     <link name="${prefix}left_wheel">
       <collision>
-        <origin xyz="0 0 0" rpy="${PI/2} 0 0"/>
+        <origin xyz="0 0 0" rpy="0 0 0"/>
         <geometry>
           <cylinder length="${wheel_len}" radius="${wheel_radius}"/>
@@ -58,5 +62,5 @@
       </collision>
       <visual>
-        <origin xyz="0 0 0" rpy="${PI/2} 0 0"/>
+        <origin xyz="0 0 0" rpy="0 0 0"/>
         <geometry>
           <cylinder length="${wheel_len}" radius="${wheel_radius}"/>
@@ -64,17 +68,10 @@
         <material name="black"/>
       </visual>
-      <inertial>
-        <origin xyz="0 0 0" rpy="${PI/2} 0 0"/>
-        <mass value="${wheel_mass}"/>
-        <inertia
-          ixx="${wheel_mass / 12.0 * (3*wheel_radius + wheel_len*wheel_len)}" ixy="0.0" ixz="0.0"
-          iyy="${wheel_mass / 12.0 * wheel_radius*wheel_radius}" iyz="0.0"
-          izz="${wheel_mass / 12.0 * wheel_radius*wheel_radius}"/>
-        </inertial>
       </link>
+<!-- *********************** caster rear wheel Link *********************** -->
     <joint name="${prefix}right_wheel_joint" type="continuous">
       <parent link="${prefix}base_link"/>
       <child link="${prefix}right_wheel"/>
-      <origin xyz="0 ${wheel_offset_y} ${z_offset}" rpy="0 0 0"/>
+      <origin xyz="0  ${wheel_offset_y} ${wheel_radius}" rpy="${PI/2} 0 0"/>
       <axis xyz="0 1 0"/>
       <dynamics damping="0.2"/>
@@ -83,5 +80,5 @@
     <link name="${prefix}right_wheel">
       <collision>
-        <origin xyz="0 0 0" rpy="${PI/2} 0 0"/>
+        <origin xyz="0 0 0" rpy="0 0 0"/>
         <geometry>
           <cylinder length="${wheel_len}" radius="${wheel_radius}"/>
@@ -89,5 +86,5 @@
       </collision>
       <visual>
-        <origin xyz="0 0 0" rpy="${PI/2} 0 0"/>
+        <origin xyz="0 0 0" rpy="0 0 0"/>
         <geometry>
           <cylinder length="${wheel_len}" radius="${wheel_radius}"/>
@@ -95,19 +92,11 @@
         <material name="black"/>
       </visual>
-      <inertial>
-        <origin xyz="0 0 0" rpy="${PI/2} 0 0"/>
-        <mass value="${wheel_mass}"/>
-        <inertia
-          ixx="${wheel_mass / 12.0 * (3*wheel_radius + wheel_len*wheel_len)}" ixy="0.0" ixz="0.0"
-          iyy="${wheel_mass / 12.0 * wheel_radius*wheel_radius}" iyz="0.0"
-          izz="${wheel_mass / 12.0 * wheel_radius*wheel_radius}"/>
-        </inertial>
       </link>
+    <!-- *********************** caster rear wheel Link *********************** -->
     <joint name="${prefix}caster_rear_wheel_joint" type="fixed">
       <parent link="${prefix}base_link"/>
       <child link="${prefix}caster_rear_wheel"/>
-      <origin xyz="${-base_width + caster_wheel_radius} 0 ${z_offset}" rpy="0 0 0"/>
+      <origin xyz="${-base_width + caster_wheel_radius} 0 ${caster_wheel_radius}" rpy="0 0 0"/>
     </joint>
-    <!-- caster rear wheel Link -->
     <link name="${prefix}caster_rear_wheel">
       <collision>
@@ -133,4 +122,27 @@
         </inertial>
       </link>
+  <!-- *********************** LIDAR SETUP **********************************  -->
+  <joint name="lidar_joint" type="fixed">
+    <parent link="base_link"/>
+    <child link="lidar_link"/>
+    <origin xyz="-.120 0 .080" rpy="0 0 0"/>
+  </joint>
+  <link name="lidar_link">
+    <collision>
+     <origin xyz="0 0 0" rpy="0 0 0"/>
+     <geometry>
+      <cylinder radius="0.0508" length="0.080"/>
+     </geometry>
+    </collision>
+    <visual>
+     <origin xyz="0 0 0" rpy="0 0 0"/>
+     <geometry>
+      <cylinder radius="0.0508" length="0.08"/>
+     </geometry>
+     <material name="Black">
+          <color rgba="${0/255} ${0/255} ${0/255} 1.0"/>
+     </material>
+    </visual>
+  </link>
   </xacro:macro>
 </robot>

Commit message: clean up

File: ros2_control_demo_description/diffbot_description/urdf/diffbot_description.urdf.xacro (robot description, xacro)
@@ -2,6 +2,6 @@
 <robot xmlns:xacro="http://www.ros.org/wiki/xacro">
   <xacro:macro name="diffbot" params="prefix">
-  <xacro:include filename="/home/mg/ros2_ddws/install/realsense2_description/share/realsense2_description/urdf/_d435i.urdf.xacro"/>
-  <xacro:include filename="/home/mg/ros2_ddws/install/realsense2_description/share/realsense2_description/urdf/_d435i_imu_modules.urdf.xacro"/>
+  <xacro:include filename="/home/mg/ws2/install/realsense2_description/share/realsense2_description/urdf/_d435i.urdf.xacro"/>
+  <xacro:include filename="/home/mg/ws2/install/realsense2_description/share/realsense2_description/urdf/_d435i_imu_modules.urdf.xacro"/>
   <!-- Constants for robot dimensions -->
   <xacro:property name="PI" value="3.1415926535897931"/>
@@ -18,13 +18,6 @@
   <xacro:property name="z_offset" value="-${base_height/2}" /> <!-- Space btw top of beam and the each joint -->
   <!-- *********************** Base Link *********************** -->
-  <link name="${prefix}base_link">
-  </link>
-      <joint name="${prefix}base_joint" type="fixed">
-      <parent link="${prefix}base_link"/>
-      <child link="${prefix}base_platform"/>
-      <origin xyz="${-base_length/2} 0 ${wheel_radius}" rpy="0 0 0"/>
-      <axis xyz="0 0 0"/>
-    </joint>
-    <link name="${prefix}base_platform">
+  <link name="${prefix}base_link"/>
+  <link name="${prefix}base_footprint">
       <collision>
         <origin xyz="0 0 0" rpy="0 0 0"/>
@@ -33,12 +26,11 @@
         </geometry>
       </collision>
-      <visual>
-        <origin xyz="0 0 0" rpy="0 0 0"/>
-        <geometry>
-          <box size="${base_length} ${base_width} ${base_height}"/>
-        </geometry>
-        <material name="orange"/>
-      </visual>
     </link>
+  <joint name="${prefix}base_joint" type="fixed">
+      <parent link="${prefix}base_link"/>
+      <child link="${prefix}base_footprint"/>
+      <origin xyz="${-base_length/2} 0 ${wheel_radius}" rpy="0 0 0"/>
+      <axis xyz="0 0 0"/>
+  </joint>
 <!-- *********************** d435i *********************** -->
   <xacro:sensor_d435i parent="base_link" use_nominal_extrinsics="false">
@@ -125,8 +117,8 @@
   <joint name="lidar_joint" type="fixed">
     <parent link="base_link"/>
-    <child link="lidar_link"/>
+    <child link="base_scan"/>
     <origin xyz="-.120 0 .080" rpy="0 0 0"/>
   </joint>
-  <link name="lidar_link">
+  <link name="base_scan">
     <collision>
      <origin xyz="0 0 0" rpy="0 0 0"/>

Commit message: gdfs

File: ros2_control_demo_description/diffbot_description/urdf/diffbot_description.urdf.xacro (robot description, xacro)
@@ -118,5 +118,5 @@
     <parent link="base_link"/>
     <child link="base_scan"/>
-    <origin xyz="-.120 0 .080" rpy="0 0 0"/>
+    <origin xyz="-.120 0 .080" rpy="0 0 ${PI}"/>
   </joint>
   <link name="base_scan">

Commit message: realsense working, diffdrive hang

File: ros2_control_demo_description/diffbot_description/urdf/diffbot_description.urdf.xacro (robot description, xacro)
@@ -1,4 +1,4 @@
 <?xml version="1.0"?>
-<robot xmlns:xacro="http://www.ros.org/wiki/xacro">
+<robot xmlns:xacro="http://www.ros.org/wiki/xacro" name="diffbot">
   <xacro:macro name="diffbot" params="prefix">
   <xacro:include filename="/home/mg/ws2/install/realsense2_description/share/realsense2_description/urdf/_d435i.urdf.xacro"/>
@@ -17,6 +17,5 @@
   <xacro:property name="caster_wheel_radius" value="0.033" />
   <xacro:property name="z_offset" value="-${base_height/2}" /> <!-- Space btw top of beam and the each joint -->
-  <!-- *********************** Base Link *********************** -->
-  <link name="${prefix}base_link"/>
+  <!-- base footprint-->
   <link name="${prefix}base_footprint">
       <collision>
@@ -28,9 +27,11 @@
     </link>
   <joint name="${prefix}base_joint" type="fixed">
-      <parent link="${prefix}base_link"/>
-      <child link="${prefix}base_footprint"/>
+      <parent link="${prefix}base_footprint"/>
+      <child link="${prefix}base_link"/>
       <origin xyz="${-base_length/2} 0 ${wheel_radius}" rpy="0 0 0"/>
       <axis xyz="0 0 0"/>
   </joint>
+  <!-- *********************** Base Link *********************** -->
+  <link name="${prefix}base_link"/>
 <!-- *********************** d435i *********************** -->
   <xacro:sensor_d435i parent="base_link" use_nominal_extrinsics="false">
@@ -137,4 +138,60 @@
     </visual>
   </link>
+  <gazebo reference="base_scan">
+    <sensor type="ray" name="head_rplidar_sensor">
+      <pose>0 0 0 0 0 0</pose>
+      <visualize>true</visualize>
+      <update_rate>10</update_rate>
+      <ray>
+        <scan>
+          <horizontal>
+            <samples>3000</samples><!-- 0.12 degrees -->
+            <min_angle>-3.14</min_angle>
+            <max_angle>3.14</max_angle>
+          </horizontal>
+        </scan>
+        <range>
+          <min>0.15</min>
+          <max>6.0</max>
+          <resolution>0.01</resolution>
+        </range>
+        <noise>
+          <type>gaussian</type>
+          <mean>0.0</mean>
+          <stddev>0.01</stddev>
+        </noise>
+      </ray>
+      <plugin name="gazebo_ros_head_rplidar_controller" filename="libgazebo_ros_laser.so">
+        <topicName>scan</topicName>
+        <frameName>base_scan</frameName>
+      </plugin>
+    </sensor>
+  </gazebo>
+  <gazebo>
+         <plugin name="diffbot_diff_drive" filename="libgazebo_ros_diff_drive.so">
+      <ros>
+        <!-- <namespace>/tb3</namespace> -->
+      </ros>
+      <update_rate>30</update_rate>
+      <!-- wheels -->
+      <left_joint>left_wheel_joint</left_joint>
+      <right_joint>right_Wheel_joint</right_joint>
+      <!-- kinematics -->
+      <wheel_separation>0.287</wheel_separation>
+      <wheel_diameter>0.111</wheel_diameter>
+      <!-- limits -->
+      <max_wheel_torque>20</max_wheel_torque>
+      <max_wheel_acceleration>1.0</max_wheel_acceleration>
+      <command_topic>cmd_vel</command_topic>
+      <!-- output -->
+      <publish_odom>true</publish_odom>
+      <publish_odom_tf>true</publish_odom_tf>
+      <publish_wheel_tf>false</publish_wheel_tf>
+      <odometry_topic>odom</odometry_topic>
+      <odometry_frame>odom</odometry_frame>
+      <robot_base_frame>base_footprint</robot_base_frame>
+      <publishWheelJointState>true</publishWheelJointState>
+    </plugin>
+    </gazebo>
   </xacro:macro>
 </robot>

Commit message: Revert "gdfs"
This reverts commit aaf449fff3b303f9055d8505368ddc5cb4ca6882.

File: ros2_control_demo_description/diffbot_description/urdf/diffbot_description.urdf.xacro (robot description, xacro)
@@ -119,5 +119,5 @@
     <parent link="base_link"/>
     <child link="base_scan"/>
-    <origin xyz="-.120 0 .080" rpy="0 0 ${PI}"/>
+    <origin xyz="-.120 0 .080" rpy="0 0 0"/>
   </joint>
   <link name="base_scan">

Commit message: functional gazebo w 435 and stvl obstacle

File: ros2_control_demo_description/diffbot_description/urdf/diffbot_description.urdf.xacro (robot description, xacro)
@@ -3,4 +3,5 @@
   <xacro:macro name="diffbot" params="prefix">
   <xacro:include filename="/home/mg/ws2/install/realsense2_description/share/realsense2_description/urdf/_d435i.urdf.xacro"/>
+  <xacro:include filename="/home/mg/ws2/install/realsense2_description/share/realsense2_description/urdf/_d435.urdf.xacro"/>
   <xacro:include filename="/home/mg/ws2/install/realsense2_description/share/realsense2_description/urdf/_d435i_imu_modules.urdf.xacro"/>
   <!-- Constants for robot dimensions -->
@@ -35,7 +36,7 @@
   <link name="${prefix}base_link"/>
 <!-- *********************** d435i *********************** -->
-  <xacro:sensor_d435i parent="base_link" use_nominal_extrinsics="false">
+  <xacro:sensor_d435 parent="base_link" use_nominal_extrinsics="false">
     <origin xyz="0 0 ${wheel_radius}" rpy="0 0 0"/>
-  </xacro:sensor_d435i>
+  </xacro:sensor_d435>
 <!-- *********************** caster rear wheel Link *********************** -->
     <joint name="${prefix}left_wheel_joint" type="continuous">

File: ros2_control_demo_description/diffbot_description/urdf/two_wheeled_robot_nav2.urdf (robot description, URDF)
Before this commit: robot two_wheeled_robot, 5 links, 4 joints
Links:
- link base_footprint: geometry visual box size=${base_length+.08} ${base_width} 0.05
- link front_caster: geometry collision sphere radius=${(wheel_zoff)}; visual sphere radius=${(wheel_zoff)}
- link imu_link: geometry collision box size=0.01 0.01 0.01; visual box size=0.01 0.01 0.01
- link lidar_link: geometry collision cylinder length=0.06 radius=0.0508; visual cylinder length=0.06 radius=0.0508
Joints:
- joint base_joint: origin xyz=0.0 0.0 ${-(wheel_radius+wheel_zoff)} rpy=0 0 0 -> xyz=${-base_length/2} 0.0 0.0 rpy=0 0 0
- joint caster_joint: origin xyz=${caster_xoff} 0.0 ${-(base_height/2)} rpy=0 0 0 -> xyz=${-caster_xoff} 0.0 ${-(wheel_radius)} rpy=0 0 0
- joint imu_joint: origin xyz=0 0 0.01 -> xyz=0.05 0 ${wheel_radius}
- joint lidar_joint: origin xyz=0.015 0.0 0.10 rpy=0 0 0 -> xyz=-0.09 0.0 ${base_height + .015} rpy=0 0 0
